Commit message: 1.0.0.20240603212941

File: pointfoot/xacro/robot.xacro (robot description, xacro)
@@ -26,5 +26,5 @@
         </visual>
         <collision>
-            <origin rpy="0 0 0" xyz="0 0 ${base_height}/2"/>
+            <origin rpy="0 0 0" xyz="0 0 ${base_height/2}"/>
             <geometry>
                 <box size="${base_length} ${base_width} ${base_height}"/>
