Commit message: 1.0.0.20240604193954

File: pointfoot/xacro/leg.xacro (robot description, xacro)
@@ -73,5 +73,5 @@
             <parent link="hip_${name}_Link"/>
             <child link="knee_${name}_Link"/>
-            <axis xyz="0 ${mirror} 0"/>
+            <axis xyz="0 ${-mirror} 0"/>
             <dynamics damping="${damping}" friction="${friction}"/>
             <xacro:if value="${(mirror_STL == True)}">

File: pointfoot/xacro/ros2_control_interface.xacro (robot description, xacro)
@@ -9,6 +9,6 @@
                 </command_interface>
                 <command_interface name="velocity">
-                    <param name="min">-15</param>
-                    <param name="max">15</param>
+                    <param name="min">-20</param>
+                    <param name="max">20</param>
                 </command_interface>
                 <command_interface name="effort">
@@ -32,6 +32,6 @@
                 </command_interface>
                 <command_interface name="velocity">
-                    <param name="min">-15</param>
-                    <param name="max">15</param>
+                    <param name="min">-20</param>
+                    <param name="max">20</param>
                 </command_interface>
                 <command_interface name="effort">
@@ -55,6 +55,6 @@
                 </command_interface>
                 <command_interface name="velocity">
-                    <param name="min">-15</param>
-                    <param name="max">15</param>
+                    <param name="min">-20</param>
+                    <param name="max">20</param>
                 </command_interface>
                 <command_interface name="effort">
@@ -80,6 +80,6 @@
                 </command_interface>
                 <command_interface name="velocity">
-                    <param name="min">-15</param>
-                    <param name="max">15</param>
+                    <param name="min">-20</param>
+                    <param name="max">20</param>
                 </command_interface>
                 <command_interface name="effort">
@@ -103,6 +103,6 @@
                 </command_interface>
                 <command_interface name="velocity">
-                    <param name="min">-15</param>
-                    <param name="max">15</param>
+                    <param name="min">-20</param>
+                    <param name="max">20</param>
                 </command_interface>
                 <command_interface name="effort">
@@ -126,6 +126,6 @@
                 </command_interface>
                 <command_interface name="velocity">
-                    <param name="min">-15</param>
-                    <param name="max">15</param>
+                    <param name="min">-20</param>
+                    <param name="max">20</param>
                 </command_interface>
                 <command_interface name="effort">
