Commit message: 1.1.5.20240911214250

File: pointfoot/PF_P441B/urdf/robot.urdf (robot description, URDF)
Before this commit: robot point_foot, 12 links, 11 joints
Links:
- link abad_L_Link: mass 1.622 -> 1.59
- link abad_R_Link: mass 1.622 -> 1.59
- link base_Link: mass 8.996 -> 8.49; geometry collision box size=0.28 0.24 0.14; visual mesh filename=package://robot_description/pointfoot/PF_P441B/meshes/base_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
- link foot_L_Link: mass 0.176 -> 0.16
- link foot_R_Link: mass 0.176 -> 0.16
- link hip_L_Link: mass 2.401 -> 2.39; geometry collision cylinder length=0.15 radius=0.025; visual mesh filename=package://robot_description/pointfoot/PF_P441B/meshes/hip_L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
- link hip_R_Link: mass 2.401 -> 2.39; geometry collision cylinder length=0.15 radius=0.025; visual mesh filename=package://robot_description/pointfoot/PF_P441B/meshes/hip_R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
- link knee_L_Link: mass 0.558 -> 0.38
- link knee_R_Link: mass 0.558 -> 0.38
Joints:
- joint abad_L_Joint: limit lower=-0.38397 upper=1.39626 effort=80.0 velocity=20.0 -> lower=-0.38397 upper=1.39626 effort=80.0 velocity=15.0; origin xyz=0.00420 0.10500 -0.09876 rpy=0 0 0 -> xyz=16.2E-03 105E-03 -90.76E-03 rpy=0 0 0
- joint abad_R_Joint: limit lower=-1.39626 upper=0.38397 effort=80.0 velocity=20.0 -> lower=-1.39626 upper=0.38397 effort=80.0 velocity=15.0; origin xyz=0.00420 -0.10500 -0.09876 rpy=0 0 0 -> xyz=16.2E-03 -105E-03 -90.76E-03 rpy=0 0 0
- joint foot_L_Joint: origin xyz=0.14929 0 -0.26014 rpy=0 0 0 -> xyz=0.150 0 -0.2598 rpy=0 0 0
- joint foot_R_Joint: origin xyz=0.14929 0 -0.26014 rpy=0 0 0 -> xyz=0.150 0 -0.2598 rpy=0 0 0
- joint hip_L_Joint: limit lower=-1.012291 upper=1.396263 effort=80.0 velocity=20.0 -> lower=-1.012291 upper=1.396263 effort=80.0 velocity=15.0; origin xyz=-0.077 0.02050 0 rpy=0 0 0 -> xyz=-77E-03 20.5E-03 0 rpy=0 0 0
- joint hip_R_Joint: limit lower=-1.396263 upper=1.012291 effort=80.0 velocity=20.0 -> lower=-1.396263 upper=1.012291 effort=80.0 velocity=15.0; origin xyz=-0.077 -0.02050 0 rpy=0 0 0 -> xyz=-77E-03 -20.5E-03 0 rpy=0 0 0
- joint knee_L_Joint: limit lower=-0.872665 upper=1.361357 effort=80 velocity=20 -> lower=-0.872665 upper=1.361357 effort=80 velocity=15; origin xyz=-0.1500 -0.02050 -0.25981 rpy=0 0 0 -> xyz=-150E-03 -20.5E-03 -0.25981 rpy=0 0 0
- joint knee_R_Joint: limit lower=-1.361357 upper=0.872665 effort=80 velocity=20 -> lower=-1.361357 upper=0.872665 effort=80 velocity=15; origin xyz=-0.1500 0.02050 -0.25981 rpy=0 0 0 -> xyz=-150E-03 20.5E-03 -0.25981 rpy=0 0 0

File: pointfoot/PF_P441C/urdf/robot.urdf (robot description, URDF)
Before this commit: robot point_foot, 12 links, 11 joints
Links:
- link abad_L_Link: mass 1.622 -> 1.560
- link abad_R_Link: mass 1.622 -> 1.560
- link base_Link: mass 8.996 -> 9.567; geometry collision box size=0.25 0.26 0.18; visual mesh filename=package://robot_description/pointfoot/PF_P441C/meshes/base_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
- link foot_L_Link: mass 0.176 -> 0.197
- link hip_L_Link: mass 2.401 -> 2.388; geometry collision cylinder length=0.18 radius=0.035; visual mesh filename=package://robot_description/pointfoot/PF_P441C/meshes/hip_L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
- link hip_R_Link: mass 2.401 -> 2.388; geometry collision cylinder length=0.18 radius=0.035; visual mesh filename=package://robot_description/pointfoot/PF_P441C/meshes/hip_R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
- link knee_L_Link: mass 0.558 -> 0.496
- link knee_R_Link: mass 0.558 -> 0.496
Joints:
- joint abad_L_Joint: limit lower=-0.38397 upper=1.39626 effort=80.0 velocity=20.0 -> lower=-0.38397 upper=1.39626 effort=80.0 velocity=15.0; origin xyz=0.00420 0.10500 -0.09876 rpy=0 0 0 -> xyz=0.039 0.1095 -0.08725 rpy=0 0 0
- joint abad_R_Joint: limit lower=-1.39626 upper=0.38397 effort=80.0 velocity=20.0 -> lower=-1.39626 upper=0.38397 effort=80.0 velocity=15.0; origin xyz=0.00420 -0.10500 -0.09876 rpy=0 0 0 -> xyz=0.039 -0.1095 -0.08725 rpy=0 0 0
- joint foot_L_Joint: origin xyz=0.14929 0 -0.26014 rpy=0 0 0 -> xyz=0.150 0 -0.25981 rpy=0 0 0
- joint foot_R_Joint: origin xyz=0.14929 0 -0.26014 rpy=0 0 0 -> xyz=0.150 0 -0.25981 rpy=0 0 0
- joint hip_L_Joint: limit lower=-1.012291 upper=1.396263 effort=80.0 velocity=20.0 -> lower=-1.012291 upper=1.396263 effort=80.0 velocity=15.0
- joint hip_R_Joint: limit lower=-1.396263 upper=1.012291 effort=80.0 velocity=20.0 -> lower=-1.396263 upper=1.012291 effort=80.0 velocity=15.0
- joint knee_L_Joint: limit lower=-0.872665 upper=1.361357 effort=80 velocity=20 -> lower=-0.872665 upper=1.361357 effort=80 velocity=15
- joint knee_R_Joint: limit lower=-1.361357 upper=0.872665 effort=80 velocity=20 -> lower=-1.361357 upper=0.872665 effort=80 velocity=15

File: pointfoot/PF_P441C2/urdf/robot.urdf (robot description, URDF)
Before this commit: robot point_foot, 12 links, 11 joints
Links:
- link abad_L_Link: mass 1.622 -> 1.48
- link abad_R_Link: mass 1.622 -> 1.560
- link base_Link: mass 8.996 -> 9.417; geometry collision box size=0.265 0.26 0.18; visual mesh filename=package://robot_description/pointfoot/PF_P441C2/meshes/base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
- link foot_L_Link: mass 0.176 -> 0.188
- link foot_R_Link: mass 0.176 -> 0.188
- link hip_L_Link: mass 2.401 -> 2.257; geometry collision cylinder length=0.18 radius=0.035; visual mesh filename=package://robot_description/pointfoot/PF_P441C2/meshes/hip_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
- link hip_R_Link: mass 2.401 -> 2.257; geometry collision cylinder length=0.18 radius=0.035; visual mesh filename=package://robot_description/pointfoot/PF_P441C2/meshes/hip_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
- link knee_L_Link: mass 0.558 -> 0.542
- link knee_R_Link: mass 0.558 -> 0.496
Joints:
- joint abad_L_Joint: limit lower=-0.38397 upper=1.39626 effort=80.0 velocity=20.0 -> lower=-0.38397 upper=1.39626 effort=80.0 velocity=15.0; origin xyz=0.00420 0.10500 -0.09876 rpy=0 0 0 -> xyz=23.76E-03 105E-03 -93.8E-03 rpy=0 0 0
- joint abad_R_Joint: limit lower=-1.39626 upper=0.38397 effort=80.0 velocity=20.0 -> lower=-1.39626 upper=0.38397 effort=80.0 velocity=15.0; origin xyz=0.00420 -0.10500 -0.09876 rpy=0 0 0 -> xyz=23.76E-03 -105E-03 -93.8E-03 rpy=0 0 0
- joint foot_L_Joint: origin xyz=0.14929 0 -0.26014 rpy=0 0 0 -> xyz=0.150 0 -0.25981 rpy=0 0 0
- joint foot_R_Joint: origin xyz=0.14929 0 -0.26014 rpy=0 0 0 -> xyz=0.150 0 -0.25981 rpy=0 0 0
- joint hip_L_Joint: limit lower=-1.012291 upper=1.396263 effort=80.0 velocity=20.0 -> lower=-1.012291 upper=1.396263 effort=80.0 velocity=15.0
- joint hip_R_Joint: limit lower=-1.396263 upper=1.012291 effort=80.0 velocity=20.0 -> lower=-1.396263 upper=1.012291 effort=80.0 velocity=15.0
- joint knee_L_Joint: limit lower=-0.872665 upper=1.361357 effort=80 velocity=20 -> lower=-0.872665 upper=1.361357 effort=80 velocity=15
- joint knee_R_Joint: limit lower=-1.361357 upper=0.872665 effort=80 velocity=20 -> lower=-1.361357 upper=0.872665 effort=80 velocity=15
