Commit message: 1.1.5.20240919112657

File: wheellegged/WL_P311D/urdf/robot.urdf (robot description, URDF)
Before this commit: robot wheel_legged, 22 links, 21 joints
Links:
- link LF_calf: geometry collision box size=0.28 0.023 0.0451; visual mesh filename=package://robot_description/wheellegged/WL_P311D/meshes/LF_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 scale=1 1 1
- link LF_hip: geometry visual mesh filename=package://robot_description/wheellegged/WL_P311D/meshes/LF_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 scale=1 1 1
- link LF_thigh: geometry visual mesh filename=package://robot_description/wheellegged/WL_P311D/meshes/LF_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 scale=1 1 1
- link LF_wheel: geometry collision cylinder length=0.017 radius=0.127; visual mesh filename=package://robot_description/wheellegged/WL_P311D/meshes/LF_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 scale=1 1 1
- link LH_calf: geometry collision box size=0.28 0.023 0.0451; visual mesh filename=package://robot_description/wheellegged/WL_P311D/meshes/LH_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 scale=1 1 1
- link LH_hip: geometry visual mesh filename=package://robot_description/wheellegged/WL_P311D/meshes/LH_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 scale=1 1 1
- link LH_thigh: geometry visual mesh filename=package://robot_description/wheellegged/WL_P311D/meshes/LH_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 scale=1 1 1
- link LH_wheel: geometry collision cylinder length=0.017 radius=0.127; visual mesh filename=package://robot_description/wheellegged/WL_P311D/meshes/LH_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 scale=1 1 1
- link RF_calf: geometry collision box size=0.28 0.023 0.0451; visual mesh filename=package://robot_description/wheellegged/WL_P311D/meshes/RF_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 scale=1 1 1
- link RF_hip: geometry visual mesh filename=package://robot_description/wheellegged/WL_P311D/meshes/RF_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 scale=1 1 1
- link RF_thigh: geometry visual mesh filename=package://robot_description/wheellegged/WL_P311D/meshes/RF_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 scale=1 1 1
- link RF_wheel: geometry collision cylinder length=0.017 radius=0.127; visual mesh filename=package://robot_description/wheellegged/WL_P311D/meshes/RF_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 scale=1 1 1
- link RH_calf: geometry collision box size=0.28 0.023 0.0451; visual mesh filename=package://robot_description/wheellegged/WL_P311D/meshes/RH_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 scale=1 1 1
- link RH_hip: geometry visual mesh filename=package://robot_description/wheellegged/WL_P311D/meshes/RH_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 scale=1 1 1
- link RH_thigh: geometry visual mesh filename=package://robot_description/wheellegged/WL_P311D/meshes/RH_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 scale=1 1 1
- link RH_wheel: geometry collision cylinder length=0.017 radius=0.127; visual mesh filename=package://robot_description/wheellegged/WL_P311D/meshes/RH_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 scale=1 1 1
- link base: geometry collision box size=0.515 0.2635 0.151; visual mesh filename=package://robot_description/wheellegged/WL_P311D/meshes/bas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 scale=1 1 1
