Commit message: 1.1.5.20240923132101

File: pointfoot/PF_P441C2/xacro/const.xacro (robot description, xacro)
@@ -1,4 +1,4 @@
 <?xml version="1.0"?>
-<robot name="p1_description" xmlns:xacro="http://www.ros.org/wiki/xacro">
+<robot name="pointfoot" xmlns:xacro="http://www.ros.org/wiki/xacro">
     <!-- Constants for robot dimensions -->
     <xacro:property name="PI" value="3.1415926535897931"/>
@@ -6,9 +6,9 @@
     <!-- simplified collision value -->
     <xacro:property name="base_width" value="0.26"/>
-    <xacro:property name="base_length" value="0.37"/>
-    <xacro:property name="base_height" value="0.14"/>
+    <xacro:property name="base_length" value="0.265"/>
+    <xacro:property name="base_height" value="0.18"/>
     <xacro:property name="abad_radius" value="0.05"/>
-    <xacro:property name="abad_length" value="0.05"/>
-    <xacro:property name="hip_radius" value="0.035"/>
+    <xacro:property name="abad_length" value="0.035"/>
+    <xacro:property name="hip_radius" value="0.018"/>
     <xacro:property name="hip_length" value="0.15"/>
     <xacro:property name="calf_radius" value="0.03"/>
@@ -17,7 +17,7 @@
     <!-- kinematic value -->
     <!-- abad offset from base frame value -->
-    <xacro:property name="abad_offset_x" value="0.00420"/>
-    <xacro:property name="abad_offset_y" value="0.10500"/>
-    <xacro:property name="abad_offset_z" value="-0.09876"/>
+    <xacro:property name="abad_offset_x" value="23.76E-03"/>
+    <xacro:property name="abad_offset_y" value="105E-03"/>
+    <xacro:property name="abad_offset_z" value="-93.8E-03"/>
     <!-- hip offset from abad frame value -->
     <xacro:property name="hip_offset_x" value="-0.077"/>
@@ -31,5 +31,5 @@
     <xacro:property name="foot_offset_x" value="0.14929"/>
     <xacro:property name="foot_offset_y" value="0.0"/>
-    <xacro:property name="foot_offset_z" value="-0.26014"/>
+    <xacro:property name="foot_offset_z" value="-0.2598"/>
     <!-- contact offset from abad frame value -->
     <xacro:property name="contact_offset_x" value="0.0"/>
@@ -55,68 +55,68 @@
     <!-- dynamics inertial value        total 18.508kg -->
     <!-- base_Link -->
-    <xacro:property name="base_mass" value="8.996"/>
-    <xacro:property name="base_com_x" value="-0.009836"/>
-    <xacro:property name="base_com_y" value="0.002360"/>
-    <xacro:property name="base_com_z" value="-0.015289"/>
-    <xacro:property name="base_ixx" value="0.115576"/>
-    <xacro:property name="base_ixy" value="0.001120"/>
-    <xacro:property name="base_ixz" value="0.029854"/>
-    <xacro:property name="base_iyy" value="0.103653"/>
-    <xacro:property name="base_iyz" value="-0.001176"/>
-    <xacro:property name="base_izz" value="0.106090"/>
+    <xacro:property name="base_mass" value="9.417"/>
+    <xacro:property name="base_com_x" value="0.012471"/>
+    <xacro:property name="base_com_y" value="0.000160"/>
+    <xacro:property name="base_com_z" value="0.002449"/>
+    <xacro:property name="base_ixx" value="135983.638E-06"/>
+    <xacro:property name="base_ixy" value="-66.349E-06"/>
+    <xacro:property name="base_ixz" value="29962.289E-06"/>
+    <xacro:property name="base_iyy" value="109266.825E-06"/>
+    <xacro:property name="base_iyz" value="377.121E-06"/>
+    <xacro:property name="base_izz" value="95932.388E-06"/>
     <!-- abad_Link (left) -->
-    <xacro:property name="abad_mass" value="1.622"/>
-    <xacro:property name="abad_com_x" value="-0.067850"/>
-    <xacro:property name="abad_com_y" value="0.045853"/>
-    <xacro:property name="abad_com_z" value="0.001067"/>
-    <xacro:property name="abad_ixx" value="0.001827"/>
-    <xacro:property name="abad_ixy" value="0.000453"/>
-    <xacro:property name="abad_ixz" value="-0.000010"/>
-    <xacro:property name="abad_iyy" value="0.002730"/>
-    <xacro:property name="abad_iyz" value="-0.000021"/>
-    <xacro:property name="abad_izz" value="0.002448"/>
+    <xacro:property name="abad_mass" value="1.48"/>
+    <xacro:property name="abad_com_x" value="-69.561E-03"/>
+    <xacro:property name="abad_com_y" value="44.266E-03"/>
+    <xacro:property name="abad_com_z" value="0.691E-03"/>
+    <xacro:property name="abad_ixx" value="1549.917E-06"/>
+    <xacro:property name="abad_ixy" value="389.821E-06"/>
+    <xacro:property name="abad_ixz" value="-13.288E-06"/>
+    <xacro:property name="abad_iyy" value="2365.872E-06"/>
+    <xacro:property name="abad_iyz" value="-8.79E-06"/>
+    <xacro:property name="abad_izz" value="2061.315E-06"/>
     <!-- hip_Link (left) -->
-    <xacro:property name="hip_mass" value="2.401"/>
-    <xacro:property name="hip_com_x" value="-0.029468"/>
-    <xacro:property name="hip_com_y" value="-0.045739"/>
-    <xacro:property name="hip_com_z" value="-0.041923"/>
-    <xacro:property name="hip_ixx" value="0.018353"/>
-    <xacro:property name="hip_ixy" value="0.001826"/>
-    <xacro:property name="hip_ixz" value="-0.009904"/>
-    <xacro:property name="hip_iyy" value="0.024534"/>
-    <xacro:property name="hip_iyz" value="0.002546"/>
-    <xacro:property name="hip_izz" value="0.009898"/>
+    <xacro:property name="hip_mass" value="2.257"/>
+    <xacro:property name="hip_com_x" value="-28.190E-03"/>
+    <xacro:property name="hip_com_y" value="-47.565E-03"/>
+    <xacro:property name="hip_com_z" value="-39.447E-03"/>
+    <xacro:property name="hip_ixx" value="16879.283E-06"/>
+    <xacro:property name="hip_ixy" value="1598.591E-06"/>
+    <xacro:property name="hip_ixz" value="-9277.159E-06"/>
+    <xacro:property name="hip_iyy" value="22911.064E-06"/>
+    <xacro:property name="hip_iyz" value="2157.766E-06"/>
+    <xacro:property name="hip_izz" value="9272.939E-06"/>
     <!-- knee_Link (left) -->
-    <xacro:property name="knee_mass" value="0.558"/>
-    <xacro:property name="knee_com_x" value="0.043236"/>
-    <xacro:property name="knee_com_y" value="-0.000044"/>
-    <xacro:property name="knee_com_z" value="-0.069329"/>
-    <xacro:property name="knee_ixx" value="0.003349"/>
-    <xacro:property name="knee_ixy" value="-0.000002"/>
-    <xacro:property name="knee_ixz" value="0.002081"/>
-    <xacro:property name="knee_iyy" value="0.004733"/>
-    <xacro:property name="knee_iyz" value="0.000002"/>
-    <xacro:property name="knee_izz" value="0.001480"/>
+    <xacro:property name="knee_mass" value="0.542"/>
+    <xacro:property name="knee_com_x" value="52.190E-03"/>
+    <xacro:property name="knee_com_y" value="1.499E-03"/>
+    <xacro:property name="knee_com_z" value="-82.413E-03"/>
+    <xacro:property name="knee_ixx" value="2913.171E-06"/>
+    <xacro:property name="knee_ixy" value="-7.196E-06"/>
+    <xacro:property name="knee_ixz" value="1808.624E-06"/>
+    <xacro:property name="knee_iyy" value="4151.771E-06"/>
+    <xacro:property name="knee_iyz" value="7.891E-06"/>
+    <xacro:property name="knee_izz" value="1318.752E-06"/>
     <!-- foot_Link (left) -->
-    <xacro:property name="foot_mass" value="0.176"/>
-    <xacro:property name="foot_com_x" value="-0.000739"/>
-    <xacro:property name="foot_com_y" value="0.000007"/>
-    <xacro:property name="foot_com_z" value="0.005104"/>
-    <xacro:property name="foot_ixx" value="0.000095"/>
-    <xacro:property name="foot_ixy" value="0.0"/>
-    <xacro:property name="foot_ixz" value="0.000004"/>
-    <xacro:property name="foot_iyy" value="0.000096"/>
-    <xacro:property name="foot_iyz" value="0.0"/>
-    <xacro:property name="foot_izz" value="0.000071"/>
+    <xacro:property name="foot_mass" value="0.188"/>
+    <xacro:property name="foot_com_x" value="-0.892E-03"/>
+    <xacro:property name="foot_com_y" value="-0.005E-03"/>
+    <xacro:property name="foot_com_z" value="5.152E-03"/>
+    <xacro:property name="foot_ixx" value="99.487E-06"/>
+    <xacro:property name="foot_ixy" value="-0.035E-06"/>
+    <xacro:property name="foot_ixz" value="4.098E-06"/>
+    <xacro:property name="foot_iyy" value="103.070E-06"/>
+    <xacro:property name="foot_iyz" value="-0.013E-06"/>
+    <xacro:property name="foot_izz" value="79.322E-06"/>
     <!-- contact_Link (left) -->
     <xacro:property name="contact_mass" value="1e-6"/>
     <xacro:property name="contact_com_x" value="-6.4629E-05"/>
     <xacro:property name="contact_com_y" value="5.464E-05"/>
-    <xacro:property name="contact_com_z" value="0.005104"/>
-    <xacro:property name="contact_ixx" value="0.000095"/>
+    <xacro:property name="contact_com_z" value="0.0011936"/>
+    <xacro:property name="contact_ixx" value="1e-12"/>
     <xacro:property name="contact_ixy" value="0.0"/>
     <xacro:property name="contact_ixz" value="0.000004"/>
-    <xacro:property name="contact_iyy" value="0.000096"/>
+    <xacro:property name="contact_iyy" value="1e-12"/>
     <xacro:property name="contact_iyz" value="0.0"/>
-    <xacro:property name="contact_izz" value="0.000071"/>
+    <xacro:property name="contact_izz" value="1e-12"/>
 </robot>
