Commit message: 1.1.5.20241105095313

File: pointfoot/PF_TRON1A/xacro/leg.xacro (robot description, xacro)
@@ -1,5 +1,5 @@
 <?xml version="1.0"?>
 <robot xmlns:xacro="http://www.ros.org/wiki/xacro">
-    <xacro:include filename="$(find robot_description)/pointfoot/PF_P441C2/xacro/transmission.xacro"/>
+    <xacro:include filename="$(find robot_description)/pointfoot/PF_TRON1A/xacro/transmission.xacro"/>
     <xacro:macro name="leg" params="name mirror mirror_STL *origin">
         <joint name="abad_${name}_joint" type="revolute">
@@ -22,5 +22,5 @@
                 <origin rpy="0 0 0" xyz="0 0 0"/>
                 <geometry>
-                    <mesh filename="$(find robot_description)/pointfoot/PF_P441C2/meshes/abad_${name}_Link.STL" scale="1 1 1"/>
+                    <mesh filename="$(find robot_description)/pointfoot/PF_TRON1A/meshes/abad_${name}_Link.STL" scale="1 1 1"/>
                 </geometry>
                 <material name="black"/>
@@ -54,5 +54,5 @@
                 <origin rpy="0 0 0" xyz="0 0 0"/>
                 <geometry>
-                    <mesh filename="$(find robot_description)/pointfoot/PF_P441C2/meshes/hip_${name}_Link.STL" scale="1 1 1"/>
+                    <mesh filename="$(find robot_description)/pointfoot/PF_TRON1A/meshes/hip_${name}_Link.STL" scale="1 1 1"/>
                 </geometry>
                 <material name="black"/>
@@ -86,5 +86,5 @@
                 <origin rpy="0 0 0" xyz="0 0 0"/>
                 <geometry>
-                    <mesh filename="$(find robot_description)/pointfoot/PF_P441C2/meshes/knee_${name}_Link.STL" scale="1 1 1"/>
+                    <mesh filename="$(find robot_description)/pointfoot/PF_TRON1A/meshes/knee_${name}_Link.STL" scale="1 1 1"/>
                 </geometry>
                 <material name="black"/>
@@ -118,5 +118,5 @@
                 <origin rpy="0 0 0" xyz="0 0 0"/>
                 <geometry>
-                    <mesh filename="$(find robot_description)/pointfoot/PF_P441C2/meshes/foot_${name}_Link.STL" scale="1 1 1"/>
+                    <mesh filename="$(find robot_description)/pointfoot/PF_TRON1A/meshes/foot_${name}_Link.STL" scale="1 1 1"/>
                 </geometry>
                 <material name="grey"/>
@@ -148,5 +148,5 @@
                 <origin rpy="0 0 0" xyz="0 0 0"/>
                 <geometry>
-                    <mesh filename="$(find robot_description)/pointfoot/PF_P441C2/meshes/foot_${name}_Link.STL" scale="1 1 1"/>
+                    <mesh filename="$(find robot_description)/pointfoot/PF_TRON1A/meshes/foot_${name}_Link.STL" scale="1 1 1"/>
                 </geometry>
                 <material name="grey"/>

File: pointfoot/PF_TRON1A/xacro/robot.xacro (robot description, xacro)
@@ -3,9 +3,9 @@
     <xacro:arg name="use_gazebo" default="false"/>
     <xacro:arg name="use_support" default="false"/>
-    <xacro:include filename="$(find robot_description)/pointfoot/PF_P441C2/xacro/const.xacro"/>
-    <xacro:include filename="$(find robot_description)/pointfoot/PF_P441C2/xacro/materials.xacro"/>
-    <xacro:include filename="$(find robot_description)/pointfoot/PF_P441C2/xacro/leg.xacro"/>
-    <xacro:include filename="$(find robot_description)/pointfoot/PF_P441C2/xacro/gazebo.xacro"/>
-    <xacro:include filename="$(find robot_description)/pointfoot/PF_P441C2/xacro/ros2_control_interface.xacro"/>
+    <xacro:include filename="$(find robot_description)/pointfoot/PF_TRON1A/xacro/const.xacro"/>
+    <xacro:include filename="$(find robot_description)/pointfoot/PF_TRON1A/xacro/materials.xacro"/>
+    <xacro:include filename="$(find robot_description)/pointfoot/PF_TRON1A/xacro/leg.xacro"/>
+    <xacro:include filename="$(find robot_description)/pointfoot/PF_TRON1A/xacro/gazebo.xacro"/>
+    <xacro:include filename="$(find robot_description)/pointfoot/PF_TRON1A/xacro/ros2_control_interface.xacro"/>
     <!-- Rollover Protection mode will add an additional stick on the top, use "true" or "false" to switch it. -->
     <xacro:property name="rolloverProtection" value="false"/>
@@ -23,5 +23,5 @@
             <origin rpy="0 0 0" xyz="0 0 0"/>
             <geometry>
-                <mesh filename="$(find robot_description)/pointfoot/PF_P441C2/meshes/base_Link.STL" scale="1 1 1"/>
+                <mesh filename="$(find robot_description)/pointfoot/PF_TRON1A/meshes/base_Link.STL" scale="1 1 1"/>
             </geometry>
             <material name="orange"/>

File: pointfoot/SF_TRON1A/urdf/robot.urdf (robot description, URDF)
Before this commit: robot point_foot, 12 links, 11 joints
Links:
- link abad_L_Link: geometry collision cylinder length=0.05 radius=0.05; visual mesh filename=package://robot_description/pointfoot/SF_TRON1A/meshes/abad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
- link abad_R_Link: geometry collision cylinder length=0.05 radius=0.05; visual mesh filename=package://robot_description/pointfoot/SF_TRON1A/meshes/abad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
- link base_Link: geometry collision box size=0.265 0.26 0.18; visual mesh filename=package://robot_description/pointfoot/SF_TRON1A/meshes/base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
- link foot_L_Link: geometry collision sphere radius=0.032; visual mesh filename=package://robot_description/pointfoot/SF_TRON1A/meshes/foot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
- link foot_R_Link: geometry collision sphere radius=0.032; visual mesh filename=package://robot_description/pointfoot/SF_TRON1A/meshes/foot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
- link hip_L_Link: geometry collision cylinder length=0.18 radius=0.035; visual mesh filename=package://robot_description/pointfoot/SF_TRON1A/meshes/hip_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
- link hip_R_Link: geometry collision cylinder length=0.18 radius=0.035; visual mesh filename=package://robot_description/pointfoot/SF_TRON1A/meshes/hip_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
- link knee_L_Link: geometry collision cylinder length=0.26 radius=0.015; visual mesh filename=package://robot_description/pointfoot/SF_TRON1A/meshes/knee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
- link knee_R_Link: geometry collision cylinder length=0.26 radius=0.015; visual mesh filename=package://robot_description/pointfoot/SF_TRON1A/meshes/knee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

File: pointfoot/SF_TRON1A/xacro/leg.xacro (robot description, xacro)
@@ -1,5 +1,5 @@
 <?xml version="1.0"?>
 <robot xmlns:xacro="http://www.ros.org/wiki/xacro">
-    <xacro:include filename="$(find robot_description)/pointfoot/PF_P441C2/xacro/transmission.xacro"/>
+    <xacro:include filename="$(find robot_description)/pointfoot/SF_TRON1A/xacro/transmission.xacro"/>
     <xacro:macro name="leg" params="name mirror mirror_STL *origin">
         <joint name="abad_${name}_joint" type="revolute">
@@ -22,5 +22,5 @@
                 <origin rpy="0 0 0" xyz="0 0 0"/>
                 <geometry>
-                    <mesh filename="$(find robot_description)/pointfoot/PF_P441C2/meshes/abad_${name}_Link.STL" scale="1 1 1"/>
+                    <mesh filename="$(find robot_description)/pointfoot/SF_TRON1A/meshes/abad_${name}_Link.STL" scale="1 1 1"/>
                 </geometry>
                 <material name="black"/>
@@ -54,5 +54,5 @@
                 <origin rpy="0 0 0" xyz="0 0 0"/>
                 <geometry>
-                    <mesh filename="$(find robot_description)/pointfoot/PF_P441C2/meshes/hip_${name}_Link.STL" scale="1 1 1"/>
+                    <mesh filename="$(find robot_description)/pointfoot/SF_TRON1A/meshes/hip_${name}_Link.STL" scale="1 1 1"/>
                 </geometry>
                 <material name="black"/>
@@ -86,5 +86,5 @@
                 <origin rpy="0 0 0" xyz="0 0 0"/>
                 <geometry>
-                    <mesh filename="$(find robot_description)/pointfoot/PF_P441C2/meshes/knee_${name}_Link.STL" scale="1 1 1"/>
+                    <mesh filename="$(find robot_description)/pointfoot/SF_TRON1A/meshes/knee_${name}_Link.STL" scale="1 1 1"/>
                 </geometry>
                 <material name="black"/>
@@ -118,5 +118,5 @@
                 <origin rpy="0 0 0" xyz="0 0 0"/>
                 <geometry>
-                    <mesh filename="$(find robot_description)/pointfoot/PF_P441C2/meshes/foot_${name}_Link.STL" scale="1 1 1"/>
+                    <mesh filename="$(find robot_description)/pointfoot/SF_TRON1A/meshes/foot_${name}_Link.STL" scale="1 1 1"/>
                 </geometry>
                 <material name="grey"/>
@@ -148,5 +148,5 @@
                 <origin rpy="0 0 0" xyz="0 0 0"/>
                 <geometry>
-                    <mesh filename="$(find robot_description)/pointfoot/PF_P441C2/meshes/foot_${name}_Link.STL" scale="1 1 1"/>
+                    <mesh filename="$(find robot_description)/pointfoot/SF_TRON1A/meshes/foot_${name}_Link.STL" scale="1 1 1"/>
                 </geometry>
                 <material name="grey"/>

File: pointfoot/SF_TRON1A/xacro/robot.xacro (robot description, xacro)
@@ -3,9 +3,9 @@
     <xacro:arg name="use_gazebo" default="false"/>
     <xacro:arg name="use_support" default="false"/>
-    <xacro:include filename="$(find robot_description)/pointfoot/PF_P441C2/xacro/const.xacro"/>
-    <xacro:include filename="$(find robot_description)/pointfoot/PF_P441C2/xacro/materials.xacro"/>
-    <xacro:include filename="$(find robot_description)/pointfoot/PF_P441C2/xacro/leg.xacro"/>
-    <xacro:include filename="$(find robot_description)/pointfoot/PF_P441C2/xacro/gazebo.xacro"/>
-    <xacro:include filename="$(find robot_description)/pointfoot/PF_P441C2/xacro/ros2_control_interface.xacro"/>
+    <xacro:include filename="$(find robot_description)/pointfoot/SF_TRON1A/xacro/const.xacro"/>
+    <xacro:include filename="$(find robot_description)/pointfoot/SF_TRON1A/xacro/materials.xacro"/>
+    <xacro:include filename="$(find robot_description)/pointfoot/SF_TRON1A/xacro/leg.xacro"/>
+    <xacro:include filename="$(find robot_description)/pointfoot/SF_TRON1A/xacro/gazebo.xacro"/>
+    <xacro:include filename="$(find robot_description)/pointfoot/SF_TRON1A/xacro/ros2_control_interface.xacro"/>
     <!-- Rollover Protection mode will add an additional stick on the top, use "true" or "false" to switch it. -->
     <xacro:property name="rolloverProtection" value="false"/>
@@ -23,5 +23,5 @@
             <origin rpy="0 0 0" xyz="0 0 0"/>
             <geometry>
-                <mesh filename="$(find robot_description)/pointfoot/PF_P441C2/meshes/base_Link.STL" scale="1 1 1"/>
+                <mesh filename="$(find robot_description)/pointfoot/SF_TRON1A/meshes/base_Link.STL" scale="1 1 1"/>
             </geometry>
             <material name="orange"/>

File: pointfoot/WF_TRON1A/urdf/robot.urdf (robot description, URDF)
Before this commit: robot wheel_biped, 9 links, 8 joints
Links:
- link abad_L_Link: geometry collision cylinder length=0.05 radius=0.05; visual mesh filename=package://robot_description/pointfoot/WF_TRON1A/meshes/abad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
- link abad_R_Link: geometry collision cylinder length=0.05 radius=0.05; visual mesh filename=package://robot_description/pointfoot/WF_TRON1A/meshes/abad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
- link base_Link: geometry collision box size=0.27 0.26 0.19; visual mesh filename=package://robot_description/pointfoot/WF_TRON1A/meshes/base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
- link hip_L_Link: geometry collision cylinder length=0.15 radius=0.035; visual mesh filename=package://robot_description/pointfoot/WF_TRON1A/meshes/hip_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
- link hip_R_Link: geometry collision cylinder length=0.15 radius=0.035; visual mesh filename=package://robot_description/pointfoot/WF_TRON1A/meshes/hip_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
- link knee_L_Link: geometry collision cylinder length=0.26 radius=0.015; visual mesh filename=package://robot_description/pointfoot/WF_TRON1A/meshes/knee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
- link knee_R_Link: geometry collision cylinder length=0.26 radius=0.015; visual mesh filename=package://robot_description/pointfoot/WF_TRON1A/meshes/knee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
- link wheel_L_Link: geometry collision cylinder length=0.05 radius=0.127; visual mesh filename=package://robot_description/pointfoot/WF_TRON1A/meshes/whee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
- link wheel_R_Link: geometry collision cylinder length=0.05 radius=0.127; visual mesh filename=package://robot_description/pointfoot/WF_TRON1A/meshes/whee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

File: pointfoot/WF_TRON1A/xacro/leg.xacro (robot description, xacro)
@@ -1,5 +1,5 @@
 <?xml version="1.0"?>
 <robot xmlns:xacro="http://www.ros.org/wiki/xacro">
-    <xacro:include filename="$(find robot_description)/pointfoot/PF_P441C2/xacro/transmission.xacro"/>
+    <xacro:include filename="$(find robot_description)/pointfoot/WF_TRON1A/xacro/transmission.xacro"/>
     <xacro:macro name="leg" params="name mirror mirror_STL *origin">
         <joint name="abad_${name}_joint" type="revolute">
@@ -22,5 +22,5 @@
                 <origin rpy="0 0 0" xyz="0 0 0"/>
                 <geometry>
-                    <mesh filename="$(find robot_description)/pointfoot/PF_P441C2/meshes/abad_${name}_Link.STL" scale="1 1 1"/>
+                    <mesh filename="$(find robot_description)/pointfoot/WF_TRON1A/meshes/abad_${name}_Link.STL" scale="1 1 1"/>
                 </geometry>
                 <material name="black"/>
@@ -54,5 +54,5 @@
                 <origin rpy="0 0 0" xyz="0 0 0"/>
                 <geometry>
-                    <mesh filename="$(find robot_description)/pointfoot/PF_P441C2/meshes/hip_${name}_Link.STL" scale="1 1 1"/>
+                    <mesh filename="$(find robot_description)/pointfoot/WF_TRON1A/meshes/hip_${name}_Link.STL" scale="1 1 1"/>
                 </geometry>
                 <material name="black"/>
@@ -86,5 +86,5 @@
                 <origin rpy="0 0 0" xyz="0 0 0"/>
                 <geometry>
-                    <mesh filename="$(find robot_description)/pointfoot/PF_P441C2/meshes/knee_${name}_Link.STL" scale="1 1 1"/>
+                    <mesh filename="$(find robot_description)/pointfoot/WF_TRON1A/meshes/knee_${name}_Link.STL" scale="1 1 1"/>
                 </geometry>
                 <material name="black"/>
@@ -118,5 +118,5 @@
                 <origin rpy="0 0 0" xyz="0 0 0"/>
                 <geometry>
-                    <mesh filename="$(find robot_description)/pointfoot/PF_P441C2/meshes/foot_${name}_Link.STL" scale="1 1 1"/>
+                    <mesh filename="$(find robot_description)/pointfoot/WF_TRON1A/meshes/foot_${name}_Link.STL" scale="1 1 1"/>
                 </geometry>
                 <material name="grey"/>
@@ -148,5 +148,5 @@
                 <origin rpy="0 0 0" xyz="0 0 0"/>
                 <geometry>
-                    <mesh filename="$(find robot_description)/pointfoot/PF_P441C2/meshes/foot_${name}_Link.STL" scale="1 1 1"/>
+                    <mesh filename="$(find robot_description)/pointfoot/WF_TRON1A/meshes/foot_${name}_Link.STL" scale="1 1 1"/>
                 </geometry>
                 <material name="grey"/>

File: pointfoot/WF_TRON1A/xacro/robot.xacro (robot description, xacro)
@@ -3,9 +3,9 @@
     <xacro:arg name="use_gazebo" default="false"/>
     <xacro:arg name="use_support" default="false"/>
-    <xacro:include filename="$(find robot_description)/pointfoot/PF_P441C2/xacro/const.xacro"/>
-    <xacro:include filename="$(find robot_description)/pointfoot/PF_P441C2/xacro/materials.xacro"/>
-    <xacro:include filename="$(find robot_description)/pointfoot/PF_P441C2/xacro/leg.xacro"/>
-    <xacro:include filename="$(find robot_description)/pointfoot/PF_P441C2/xacro/gazebo.xacro"/>
-    <xacro:include filename="$(find robot_description)/pointfoot/PF_P441C2/xacro/ros2_control_interface.xacro"/>
+    <xacro:include filename="$(find robot_description)/pointfoot/WF_TRON1A/xacro/const.xacro"/>
+    <xacro:include filename="$(find robot_description)/pointfoot/WF_TRON1A/xacro/materials.xacro"/>
+    <xacro:include filename="$(find robot_description)/pointfoot/WF_TRON1A/xacro/leg.xacro"/>
+    <xacro:include filename="$(find robot_description)/pointfoot/WF_TRON1A/xacro/gazebo.xacro"/>
+    <xacro:include filename="$(find robot_description)/pointfoot/WF_TRON1A/xacro/ros2_control_interface.xacro"/>
     <!-- Rollover Protection mode will add an additional stick on the top, use "true" or "false" to switch it. -->
     <xacro:property name="rolloverProtection" value="false"/>
@@ -23,5 +23,5 @@
             <origin rpy="0 0 0" xyz="0 0 0"/>
             <geometry>
-                <mesh filename="$(find robot_description)/pointfoot/PF_P441C2/meshes/base_Link.STL" scale="1 1 1"/>
+                <mesh filename="$(find robot_description)/pointfoot/WF_TRON1A/meshes/base_Link.STL" scale="1 1 1"/>
             </geometry>
             <material name="orange"/>
