Commit message: 1.1.5.20241118092402

File: pointfoot/PF_TRON1A/xacro/const.xacro (robot description, xacro)
@@ -17,7 +17,7 @@
     <!-- kinematic value -->
     <!-- abad offset from base frame value -->
-    <xacro:property name="abad_offset_x" value="23.76E-03"/>
+    <xacro:property name="abad_offset_x" value="55.56E-03"/>
     <xacro:property name="abad_offset_y" value="105E-03"/>
-    <xacro:property name="abad_offset_z" value="-93.8E-03"/>
+    <xacro:property name="abad_offset_z" value="-260.2E-03"/>
     <!-- hip offset from abad frame value -->
     <xacro:property name="hip_offset_x" value="-0.077"/>
@@ -29,5 +29,5 @@
     <xacro:property name="knee_offset_z" value="-0.25981"/>
     <!-- foot offset from abad frame value -->
-    <xacro:property name="foot_offset_x" value="0.14929"/>
+    <xacro:property name="foot_offset_x" value="0.145"/>
     <xacro:property name="foot_offset_y" value="0.0"/>
     <xacro:property name="foot_offset_z" value="-0.2598"/>
@@ -55,58 +55,58 @@
     <!-- dynamics inertial value        total 18.508kg -->
     <!-- base_Link -->
-    <xacro:property name="base_mass" value="9.417"/>
-    <xacro:property name="base_com_x" value="0.012471"/>
-    <xacro:property name="base_com_y" value="0.000160"/>
-    <xacro:property name="base_com_z" value="0.002449"/>
-    <xacro:property name="base_ixx" value="135983.638E-06"/>
-    <xacro:property name="base_ixy" value="-66.349E-06"/>
-    <xacro:property name="base_ixz" value="29962.289E-06"/>
-    <xacro:property name="base_iyy" value="109266.825E-06"/>
-    <xacro:property name="base_iyz" value="377.121E-06"/>
-    <xacro:property name="base_izz" value="95932.388E-06"/>
+    <xacro:property name="base_mass" value="9.585"/>
+    <xacro:property name="base_com_x" value="0.04576"/>
+    <xacro:property name="base_com_y" value="0.00014"/>
+    <xacro:property name="base_com_z" value="-0.16398"/>
+    <xacro:property name="base_ixx" value="140110.479E-06"/>
+    <xacro:property name="base_ixy" value="534.939E-06"/>
+    <xacro:property name="base_ixz" value="28184.116E-06"/>
+    <xacro:property name="base_iyy" value="110641.449E-06"/>
+    <xacro:property name="base_iyz" value="-27.278E-06"/>
+    <xacro:property name="base_izz" value="98944.542E-06"/>
     <!-- abad_Link (left) -->
-    <xacro:property name="abad_mass" value="1.48"/>
-    <xacro:property name="abad_com_x" value="-69.561E-03"/>
-    <xacro:property name="abad_com_y" value="44.266E-03"/>
-    <xacro:property name="abad_com_z" value="0.691E-03"/>
-    <xacro:property name="abad_ixx" value="1549.917E-06"/>
-    <xacro:property name="abad_ixy" value="389.821E-06"/>
-    <xacro:property name="abad_ixz" value="-13.288E-06"/>
-    <xacro:property name="abad_iyy" value="2365.872E-06"/>
-    <xacro:property name="abad_iyz" value="-8.79E-06"/>
-    <xacro:property name="abad_izz" value="2061.315E-06"/>
+    <xacro:property name="abad_mass" value="1.469"/>
+    <xacro:property name="abad_com_x" value="-69.77E-03"/>
+    <xacro:property name="abad_com_y" value="44.79E-03"/>
+    <xacro:property name="abad_com_z" value="0.57E-03"/>
+    <xacro:property name="abad_ixx" value="1555.384E-06"/>
+    <xacro:property name="abad_ixy" value="397.78E-06"/>
+    <xacro:property name="abad_ixz" value="-13.10E-06"/>
+    <xacro:property name="abad_iyy" value="2359.25E-06"/>
+    <xacro:property name="abad_iyz" value="-0.98E-06"/>
+    <xacro:property name="abad_izz" value="2080.92E-06"/>
     <!-- hip_Link (left) -->
-    <xacro:property name="hip_mass" value="2.257"/>
-    <xacro:property name="hip_com_x" value="-28.190E-03"/>
-    <xacro:property name="hip_com_y" value="-47.565E-03"/>
-    <xacro:property name="hip_com_z" value="-39.447E-03"/>
-    <xacro:property name="hip_ixx" value="16879.283E-06"/>
-    <xacro:property name="hip_ixy" value="1598.591E-06"/>
-    <xacro:property name="hip_ixz" value="-9277.159E-06"/>
-    <xacro:property name="hip_iyy" value="22911.064E-06"/>
-    <xacro:property name="hip_iyz" value="2157.766E-06"/>
-    <xacro:property name="hip_izz" value="9272.939E-06"/>
+    <xacro:property name="hip_mass" value="2.3"/>
+    <xacro:property name="hip_com_x" value="-28.69E-03"/>
+    <xacro:property name="hip_com_y" value="-47.7E-03"/>
+    <xacro:property name="hip_com_z" value="-39.92E-03"/>
+    <xacro:property name="hip_ixx" value="16937.28E-06"/>
+    <xacro:property name="hip_ixy" value="1647.03E-06"/>
+    <xacro:property name="hip_ixz" value="-9232.53E-06"/>
+    <xacro:property name="hip_iyy" value="22853.28E-06"/>
+    <xacro:property name="hip_iyz" value="2202.40E-06"/>
+    <xacro:property name="hip_izz" value="9334.19E-06"/>
     <!-- knee_Link (left) -->
-    <xacro:property name="knee_mass" value="0.542"/>
-    <xacro:property name="knee_com_x" value="52.190E-03"/>
-    <xacro:property name="knee_com_y" value="1.499E-03"/>
-    <xacro:property name="knee_com_z" value="-82.413E-03"/>
-    <xacro:property name="knee_ixx" value="2913.171E-06"/>
-    <xacro:property name="knee_ixy" value="-7.196E-06"/>
-    <xacro:property name="knee_ixz" value="1808.624E-06"/>
-    <xacro:property name="knee_iyy" value="4151.771E-06"/>
-    <xacro:property name="knee_iyz" value="7.891E-06"/>
-    <xacro:property name="knee_izz" value="1318.752E-06"/>
+    <xacro:property name="knee_mass" value="0.55"/>
+    <xacro:property name="knee_com_x" value="51.68E-03"/>
+    <xacro:property name="knee_com_y" value="1.52E-03"/>
+    <xacro:property name="knee_com_z" value="-81.48E-03"/>
+    <xacro:property name="knee_ixx" value="2949.6E-06"/>
+    <xacro:property name="knee_ixy" value="-7.86E-06"/>
+    <xacro:property name="knee_ixz" value="1830.36E-06"/>
+    <xacro:property name="knee_iyy" value="4199.48E-06"/>
+    <xacro:property name="knee_iyz" value="9.14E-06"/>
+    <xacro:property name="knee_izz" value="1330.18E-06"/>
     <!-- foot_Link (left) -->
-    <xacro:property name="foot_mass" value="0.188"/>
-    <xacro:property name="foot_com_x" value="-0.892E-03"/>
-    <xacro:property name="foot_com_y" value="-0.005E-03"/>
-    <xacro:property name="foot_com_z" value="5.152E-03"/>
-    <xacro:property name="foot_ixx" value="99.487E-06"/>
-    <xacro:property name="foot_ixy" value="-0.035E-06"/>
-    <xacro:property name="foot_ixz" value="4.098E-06"/>
-    <xacro:property name="foot_iyy" value="103.070E-06"/>
-    <xacro:property name="foot_iyz" value="-0.013E-06"/>
-    <xacro:property name="foot_izz" value="79.322E-06"/>
+    <xacro:property name="foot_mass" value="0.18"/>
+    <xacro:property name="foot_com_x" value="-1.29E-03"/>
+    <xacro:property name="foot_com_y" value="-0.01E-03"/>
+    <xacro:property name="foot_com_z" value="5.68E-03"/>
+    <xacro:property name="foot_ixx" value="97.46E-06"/>
+    <xacro:property name="foot_ixy" value="-0.04E-06"/>
+    <xacro:property name="foot_ixz" value="5.67E-06"/>
+    <xacro:property name="foot_iyy" value="99.92E-06"/>
+    <xacro:property name="foot_iyz" value="-0.01E-06"/>
+    <xacro:property name="foot_izz" value="74.7E-06"/>
     <!-- contact_Link (left) -->
     <xacro:property name="contact_mass" value="1e-6"/>

File: pointfoot/PF_TRON1A/xacro/robot.xacro (robot description, xacro)
@@ -101,3 +101,24 @@
         </gazebo>
     </xacro:if>
+    <!-- ****************************************** D435 Camera ******************************************************** -->
+    <!-- <joint name="d435_joint" type="fixed">
+        <origin rpy="0 1.063778179 0" xyz="0.13223 0.0222 -0.26826"/>
+        <parent link="base_Link"/>
+        <child link="d435_Link"/>
+    </joint>
+    <link name="d435_Link">
+        <visual>
+            <origin rpy="1.5707963267948966 0 1.5707963267948966" xyz="0.0149 -0.0175 0"/>
+            <geometry>
+                <mesh filename="package://robot_description/pointfoot/meshes_camera/d435.dae"/>
+            </geometry>
+        </visual>
+        <collision>
+            <origin rpy="0 0 0" xyz="0 -0.0175 0"/>
+            <geometry>
+                <box size="0.02505 0.09 0.025"/>
+            </geometry>
+        </collision>
+    </link> -->
+    <!-- ****************************************** D435 Camera END ******************************************************** -->
 </robot>

File: pointfoot/WF_TRON1A/urdf/robot.urdf (robot description, URDF)
Before this commit: robot wheel_biped, 10 links, 9 joints
Links:
- link abad_L_Link: mass 1.496 -> 1.469
- link abad_R_Link: mass 1.496 -> 1.469

File: pointfoot/WF_TRON1A/xacro/const.xacro (robot description, xacro)
@@ -14,10 +14,10 @@
     <xacro:property name="calf_radius" value="0.03"/>
     <xacro:property name="calf_length" value="0.26"/>
-    <xacro:property name="foot_radius" value="0.032"/>
+    <xacro:property name="wheel_radius" value="0.032"/>
     <!-- kinematic value -->
     <!-- abad offset from base frame value -->
-    <xacro:property name="abad_offset_x" value="23.76E-03"/>
+    <xacro:property name="abad_offset_x" value="55.56E-03"/>
     <xacro:property name="abad_offset_y" value="105E-03"/>
-    <xacro:property name="abad_offset_z" value="-93.8E-03"/>
+    <xacro:property name="abad_offset_z" value="-260.2E-03"/>
     <!-- hip offset from abad frame value -->
     <xacro:property name="hip_offset_x" value="-0.077"/>
@@ -28,8 +28,8 @@
     <xacro:property name="knee_offset_y" value="-0.02050"/>
     <xacro:property name="knee_offset_z" value="-0.25981"/>
-    <!-- foot offset from abad frame value -->
-    <xacro:property name="foot_offset_x" value="0.14929"/>
-    <xacro:property name="foot_offset_y" value="0.0"/>
-    <xacro:property name="foot_offset_z" value="-0.2598"/>
+    <!-- wheel offset from abad frame value -->
+    <xacro:property name="wheel_offset_x" value="0.145"/>
+    <xacro:property name="wheel_offset_y" value="0.0"/>
+    <xacro:property name="wheel_offset_z" value="-0.2598"/>
     <!-- contact offset from abad frame value -->
     <xacro:property name="contact_offset_x" value="0.0"/>
@@ -55,68 +55,57 @@
     <!-- dynamics inertial value        total 18.508kg -->
     <!-- base_Link -->
-    <xacro:property name="base_mass" value="9.417"/>
-    <xacro:property name="base_com_x" value="0.012471"/>
-    <xacro:property name="base_com_y" value="0.000160"/>
-    <xacro:property name="base_com_z" value="0.002449"/>
-    <xacro:property name="base_ixx" value="135983.638E-06"/>
-    <xacro:property name="base_ixy" value="-66.349E-06"/>
-    <xacro:property name="base_ixz" value="29962.289E-06"/>
-    <xacro:property name="base_iyy" value="109266.825E-06"/>
-    <xacro:property name="base_iyz" value="377.121E-06"/>
-    <xacro:property name="base_izz" value="95932.388E-06"/>
+    <xacro:property name="base_mass" value="9.585"/>
+    <xacro:property name="base_com_x" value="0.04576"/>
+    <xacro:property name="base_com_y" value="0.00014"/>
+    <xacro:property name="base_com_z" value="-0.16398"/>
+    <xacro:property name="base_ixx" value="140110.479E-06"/>
+    <xacro:property name="base_ixy" value="534.939E-06"/>
+    <xacro:property name="base_ixz" value="28184.116E-06"/>
+    <xacro:property name="base_iyy" value="110641.449E-06"/>
+    <xacro:property name="base_iyz" value="-27.278E-06"/>
+    <xacro:property name="base_izz" value="98944.542E-06"/>
     <!-- abad_Link (left) -->
-    <xacro:property name="abad_mass" value="1.48"/>
-    <xacro:property name="abad_com_x" value="-69.561E-03"/>
-    <xacro:property name="abad_com_y" value="44.266E-03"/>
-    <xacro:property name="abad_com_z" value="0.691E-03"/>
-    <xacro:property name="abad_ixx" value="1549.917E-06"/>
-    <xacro:property name="abad_ixy" value="389.821E-06"/>
-    <xacro:property name="abad_ixz" value="-13.288E-06"/>
-    <xacro:property name="abad_iyy" value="2365.872E-06"/>
-    <xacro:property name="abad_iyz" value="-8.79E-06"/>
-    <xacro:property name="abad_izz" value="2061.315E-06"/>
+    <xacro:property name="abad_mass" value="1.496"/>
+    <xacro:property name="abad_com_x" value="-69.77E-03"/>
+    <xacro:property name="abad_com_y" value="44.79E-03"/>
+    <xacro:property name="abad_com_z" value="0.57E-03"/>
+    <xacro:property name="abad_ixx" value="1555.384E-06"/>
+    <xacro:property name="abad_ixy" value="397.78E-06"/>
+    <xacro:property name="abad_ixz" value="-13.10E-06"/>
+    <xacro:property name="abad_iyy" value="2359.25E-06"/>
+    <xacro:property name="abad_iyz" value="-0.98E-06"/>
+    <xacro:property name="abad_izz" value="2080.92E-06"/>
     <!-- hip_Link (left) -->
-    <xacro:property name="hip_mass" value="2.257"/>
-    <xacro:property name="hip_com_x" value="-28.190E-03"/>
-    <xacro:property name="hip_com_y" value="-47.565E-03"/>
-    <xacro:property name="hip_com_z" value="-39.447E-03"/>
-    <xacro:property name="hip_ixx" value="16879.283E-06"/>
-    <xacro:property name="hip_ixy" value="1598.591E-06"/>
-    <xacro:property name="hip_ixz" value="-9277.159E-06"/>
-    <xacro:property name="hip_iyy" value="22911.064E-06"/>
-    <xacro:property name="hip_iyz" value="2157.766E-06"/>
-    <xacro:property name="hip_izz" value="9272.939E-06"/>
+    <xacro:property name="hip_mass" value="2.3"/>
+    <xacro:property name="hip_com_x" value="-28.69E-03"/>
+    <xacro:property name="hip_com_y" value="-47.7E-03"/>
+    <xacro:property name="hip_com_z" value="-39.92E-03"/>
+    <xacro:property name="hip_ixx" value="16937.28E-06"/>
+    <xacro:property name="hip_ixy" value="1647.03E-06"/>
+    <xacro:property name="hip_ixz" value="-9232.53E-06"/>
+    <xacro:property name="hip_iyy" value="22853.28E-06"/>
+    <xacro:property name="hip_iyz" value="2202.40E-06"/>
+    <xacro:property name="hip_izz" value="9334.19E-06"/>
     <!-- knee_Link (left) -->
-    <xacro:property name="knee_mass" value="0.542"/>
-    <xacro:property name="knee_com_x" value="52.190E-03"/>
-    <xacro:property name="knee_com_y" value="1.499E-03"/>
-    <xacro:property name="knee_com_z" value="-82.413E-03"/>
-    <xacro:property name="knee_ixx" value="2913.171E-06"/>
-    <xacro:property name="knee_ixy" value="-7.196E-06"/>
-    <xacro:property name="knee_ixz" value="1808.624E-06"/>
-    <xacro:property name="knee_iyy" value="4151.771E-06"/>
-    <xacro:property name="knee_iyz" value="7.891E-06"/>
-    <xacro:property name="knee_izz" value="1318.752E-06"/>
-    <!-- foot_Link (left) -->
-    <xacro:property name="foot_mass" value="0.188"/>
-    <xacro:property name="foot_com_x" value="-0.892E-03"/>
-    <xacro:property name="foot_com_y" value="-0.005E-03"/>
-    <xacro:property name="foot_com_z" value="5.152E-03"/>
-    <xacro:property name="foot_ixx" value="99.487E-06"/>
-    <xacro:property name="foot_ixy" value="-0.035E-06"/>
-    <xacro:property name="foot_ixz" value="4.098E-06"/>
-    <xacro:property name="foot_iyy" value="103.070E-06"/>
-    <xacro:property name="foot_iyz" value="-0.013E-06"/>
-    <xacro:property name="foot_izz" value="79.322E-06"/>
-    <!-- contact_Link (left) -->
-    <xacro:property name="contact_mass" value="1e-6"/>
-    <xacro:property name="contact_com_x" value="-6.4629E-05"/>
-    <xacro:property name="contact_com_y" value="5.464E-05"/>
-    <xacro:property name="contact_com_z" value="0.0011936"/>
-    <xacro:property name="contact_ixx" value="1e-12"/>
-    <xacro:property name="contact_ixy" value="0.0"/>
-    <xacro:property name="contact_ixz" value="0.000004"/>
-    <xacro:property name="contact_iyy" value="1e-12"/>
-    <xacro:property name="contact_iyz" value="0.0"/>
-    <xacro:property name="contact_izz" value="1e-12"/>
+    <xacro:property name="knee_mass" value="1.49"/>
+    <xacro:property name="knee_com_x" value="119.13E-03"/>
+    <xacro:property name="knee_com_y" value="11.06E-03"/>
+    <xacro:property name="knee_com_z" value="-203.63E-03"/>
+    <xacro:property name="knee_ixx" value="13232.8E-06"/>
+    <xacro:property name="knee_ixy" value="-435.46E-06"/>
+    <xacro:property name="knee_ixz" value="6935.69E-06"/>
+    <xacro:property name="knee_iyy" value="17661.37E-06"/>
+    <xacro:property name="knee_iyz" value="790.87E-06"/>
+    <xacro:property name="knee_izz" value="5016.98E-06"/>
+    <!-- wheel_Link (left) -->
+    <xacro:property name="wheel_mass" value="1.08"/>
+    <xacro:property name="wheel_com_x" value="0.03E-03"/>
+    <xacro:property name="wheel_com_y" value="8.07E-03"/>
+    <xacro:property name="wheel_com_z" value="-0.02E-03"/>
+    <xacro:property name="wheel_ixx" value="5155.12E-06"/>
+    <xacro:property name="wheel_ixy" value="0.01E-06"/>
+    <xacro:property name="wheel_ixz" value="-0.97E-06"/>
+    <xacro:property name="wheel_iyy" value="9742.72E-06"/>
+    <xacro:property name="wheel_iyz" value="-0.01E-06"/>
+    <xacro:property name="wheel_izz" value="5154.00E-06"/>
 </robot>

File: pointfoot/WF_TRON1A/xacro/leg.xacro (robot description, xacro)
@@ -22,5 +22,5 @@
                 <origin rpy="0 0 0" xyz="0 0 0"/>
                 <geometry>
-                    <mesh filename="$(find robot_description)/pointfoot/WF_TRON1A/meshes/abad_${name}_Link.STL" scale="1 1 1"/>
+                    <mesh filename="$(find robot_description)/pointwheel/WF_TRON1A/meshes/abad_${name}_Link.STL" scale="1 1 1"/>
                 </geometry>
                 <material name="black"/>
@@ -54,5 +54,5 @@
                 <origin rpy="0 0 0" xyz="0 0 0"/>
                 <geometry>
-                    <mesh filename="$(find robot_description)/pointfoot/WF_TRON1A/meshes/hip_${name}_Link.STL" scale="1 1 1"/>
+                    <mesh filename="$(find robot_description)/pointwheel/WF_TRON1A/meshes/hip_${name}_Link.STL" scale="1 1 1"/>
                 </geometry>
                 <material name="black"/>
@@ -86,5 +86,5 @@
                 <origin rpy="0 0 0" xyz="0 0 0"/>
                 <geometry>
-                    <mesh filename="$(find robot_description)/pointfoot/WF_TRON1A/meshes/knee_${name}_Link.STL" scale="1 1 1"/>
+                    <mesh filename="$(find robot_description)/pointwheel/WF_TRON1A/meshes/knee_${name}_Link.STL" scale="1 1 1"/>
                 </geometry>
                 <material name="black"/>
@@ -105,18 +105,18 @@
             </inertial>
         </link>
-        <joint name="foot_${name}_joint" type="fixed">
+        <joint name="wheel_${name}_joint" type="fixed">
             <origin
-                xyz="${foot_offset_x} ${foot_offset_y*mirror} ${foot_offset_z}"
+                xyz="${wheel_offset_x} ${wheel_offset_y*mirror} ${wheel_offset_z}"
                 rpy="0 0 0"/>
             <parent link="knee_${name}_Link"/>
-            <child link="foot_${name}_Link"/>
-            <axis xyz="0 ${mirror} 0"/>
+            <child link="wheel_${name}_Link"/>
+            <axis xyz="0 1 0"/>
             <dynamics damping="${damping}" friction="${friction}"/>
         </joint>
-        <link name="foot_${name}_Link">
+        <link name="wheel_${name}_Link">
             <visual>
                 <origin rpy="0 0 0" xyz="0 0 0"/>
                 <geometry>
-                    <mesh filename="$(find robot_description)/pointfoot/WF_TRON1A/meshes/foot_${name}_Link.STL" scale="1 1 1"/>
+                    <mesh filename="$(find robot_description)/pointwheel/WF_TRON1A/meshes/wheel_${name}_Link.STL" scale="1 1 1"/>
                 </geometry>
                 <material name="grey"/>
@@ -125,38 +125,14 @@
                 <origin rpy="0 0 0" xyz="0 0 0.0"/>
                 <geometry>
-                    <sphere radius="${foot_radius}"/>
+                    <sphere radius="${wheel_radius}"/>
                 </geometry>
             </collision>
             <inertial>
-                <origin rpy="0 0 0" xyz="${foot_com_x} ${foot_com_y*mirror} ${foot_com_z}"/>
-                <mass value="${foot_mass}"/>
+                <origin rpy="0 0 0" xyz="${wheel_com_x} ${wheel_com_y*mirror} ${wheel_com_z}"/>
+                <mass value="${wheel_mass}"/>
                 <inertia
-                    ixx="${foot_ixx}" ixy="${foot_ixy*mirror}" ixz="${foot_ixz}"
-                    iyy="${foot_iyy}" iyz="${foot_iyz*mirror}"
-                    izz="${foot_izz}"/>
-            </inertial>
-        </link>
-        <joint name="contact_${name}_joint" type="fixed">
-            <xacro:insert_block name="origin"/>
-            <parent link="foot_${name}_Link"/>
-            <child link="contact_${name}_Link"/>
-            <axis xyz="1 0 0"/>
-            <dynamics damping="${damping}" friction="${friction}"/>
-        </joint>
-        <link name="contact_${name}_Link">
-            <visual>
-                <origin rpy="0 0 0" xyz="0 0 0"/>
-                <geometry>
-                    <mesh filename="$(find robot_description)/pointfoot/WF_TRON1A/meshes/foot_${name}_Link.STL" scale="1 1 1"/>
-                </geometry>
-                <material name="grey"/>
-            </visual>
-            <inertial>
-                <origin rpy="0 0 0" xyz="${contact_com_x} ${contact_com_y*mirror} ${contact_com_z}"/>
-                <mass value="${contact_mass}"/>
-                <inertia
-                    ixx="${contact_ixx}" ixy="${contact_ixy*mirror}" ixz="${contact_ixz}"
-                    iyy="${contact_iyy}" iyz="${contact_iyz*mirror}"
-                    izz="${contact_izz}"/>
+                    ixx="${wheel_ixx}" ixy="${wheel_ixy*mirror}" ixz="${wheel_ixz}"
+                    iyy="${wheel_iyy}" iyz="${wheel_iyz*mirror}"
+                    izz="${wheel_izz}"/>
             </inertial>
         </link>

File: pointfoot/WF_TRON1A/xacro/robot.xacro (robot description, xacro)
@@ -101,3 +101,24 @@
         </gazebo>
     </xacro:if>
+    <!-- ****************************************** D435 Camera ******************************************************** -->
+    <!-- <joint name="d435_joint" type="fixed">
+        <origin rpy="0 1.063778179 0" xyz="0.13223 0.0222 -0.26826"/>
+        <parent link="base_Link"/>
+        <child link="d435_Link"/>
+    </joint>
+    <link name="d435_Link">
+        <visual>
+            <origin rpy="1.5707963267948966 0 1.5707963267948966" xyz="0.0149 -0.0175 0"/>
+            <geometry>
+                <mesh filename="package://robot_description/pointfoot/meshes_camera/d435.dae"/>
+            </geometry>
+        </visual>
+        <collision>
+            <origin rpy="0 0 0" xyz="0 -0.0175 0"/>
+            <geometry>
+                <box size="0.02505 0.09 0.025"/>
+            </geometry>
+        </collision>
+    </link> -->
+    <!-- ****************************************** D435 Camera END ******************************************************** -->
 </robot>
