Commit message: 1.1.5.20241119160355

File: pointfoot/PF_TRON1A/xacro/robot.xacro (robot description, xacro)
@@ -28,5 +28,5 @@
         </visual>
         <collision>
-            <origin rpy="0 0 0" xyz="0 0 ${base_height/2}"/>
+            <origin rpy="0 0 0" xyz="0.033 0 -0.07"/>
             <geometry>
                 <box size="${base_length} ${base_width} ${base_height}"/>

File: pointfoot/WF_TRON1A/xacro/const.xacro (robot description, xacro)
@@ -14,5 +14,6 @@
     <xacro:property name="calf_radius" value="0.03"/>
     <xacro:property name="calf_length" value="0.26"/>
-    <xacro:property name="wheel_radius" value="0.032"/>
+    <xacro:property name="wheel_radius" value="0.127"/>
+    <xacro:property name="wheel_length" value="0.005"/>
     <!-- kinematic value -->
     <!-- abad offset from base frame value -->
@@ -29,11 +30,7 @@
     <xacro:property name="knee_offset_z" value="-0.25981"/>
     <!-- wheel offset from abad frame value -->
-    <xacro:property name="wheel_offset_x" value="0.145"/>
-    <xacro:property name="wheel_offset_y" value="0.0"/>
-    <xacro:property name="wheel_offset_z" value="-0.2598"/>
-    <!-- contact offset from abad frame value -->
-    <xacro:property name="contact_offset_x" value="0.0"/>
-    <xacro:property name="contact_offset_y" value="0.0"/>
-    <xacro:property name="contact_offset_z" value="-0.032"/>
+    <xacro:property name="wheel_offset_x" value="0.1500"/>
+    <xacro:property name="wheel_offset_y" value="0.0435"/>
+    <xacro:property name="wheel_offset_z" value="-0.25981"/>
     <!-- joint limits -->
     <!-- <xacro:property name="damping" value="0"/> -->
@@ -53,4 +50,8 @@
     <xacro:property name="knee_velocity_max" value="15"/>
     <xacro:property name="knee_torque_max" value="80"/>
+    <xacro:property name="wheel_max" value="10000000000"/>
+    <xacro:property name="wheel_min" value="-10000000000"/>
+    <xacro:property name="wheel_velocity_max" value="40"/>
+    <xacro:property name="wheel_torque_max" value="40"/>
     <!-- dynamics inertial value        total 18.508kg -->
     <!-- base_Link -->

File: pointfoot/WF_TRON1A/xacro/leg.xacro (robot description, xacro)
@@ -22,5 +22,5 @@
                 <origin rpy="0 0 0" xyz="0 0 0"/>
                 <geometry>
-                    <mesh filename="$(find robot_description)/pointwheel/WF_TRON1A/meshes/abad_${name}_Link.STL" scale="1 1 1"/>
+                    <mesh filename="$(find robot_description)/pointfoot/WF_TRON1A/meshes/abad_${name}_Link.STL" scale="1 1 1"/>
                 </geometry>
                 <material name="black"/>
@@ -54,5 +54,5 @@
                 <origin rpy="0 0 0" xyz="0 0 0"/>
                 <geometry>
-                    <mesh filename="$(find robot_description)/pointwheel/WF_TRON1A/meshes/hip_${name}_Link.STL" scale="1 1 1"/>
+                    <mesh filename="$(find robot_description)/pointfoot/WF_TRON1A/meshes/hip_${name}_Link.STL" scale="1 1 1"/>
                 </geometry>
                 <material name="black"/>
@@ -86,5 +86,5 @@
                 <origin rpy="0 0 0" xyz="0 0 0"/>
                 <geometry>
-                    <mesh filename="$(find robot_description)/pointwheel/WF_TRON1A/meshes/knee_${name}_Link.STL" scale="1 1 1"/>
+                    <mesh filename="$(find robot_description)/pointfoot/WF_TRON1A/meshes/knee_${name}_Link.STL" scale="1 1 1"/>
                 </geometry>
                 <material name="black"/>
@@ -105,5 +105,5 @@
             </inertial>
         </link>
-        <joint name="wheel_${name}_joint" type="fixed">
+        <joint name="wheel_${name}_joint" type="revolute">
             <origin
                 xyz="${wheel_offset_x} ${wheel_offset_y*mirror} ${wheel_offset_z}"
@@ -113,4 +113,5 @@
             <axis xyz="0 1 0"/>
             <dynamics damping="${damping}" friction="${friction}"/>
+            <limit effort="${wheel_torque_max}" velocity="${wheel_velocity_max}" lower="${wheel_min*PI/180.0}" upper="${wheel_max*PI/180.0}"/>
         </joint>
         <link name="wheel_${name}_Link">
@@ -118,12 +119,12 @@
                 <origin rpy="0 0 0" xyz="0 0 0"/>
                 <geometry>
-                    <mesh filename="$(find robot_description)/pointwheel/WF_TRON1A/meshes/wheel_${name}_Link.STL" scale="1 1 1"/>
+                    <mesh filename="$(find robot_description)/pointfoot/WF_TRON1A/meshes/wheel_${name}_Link.STL" scale="1 1 1"/>
                 </geometry>
                 <material name="grey"/>
             </visual>
             <collision>
-                <origin rpy="0 0 0" xyz="0 0 0.0"/>
+                <origin rpy="1.570796327 0 0" xyz="0 ${0.008*mirror} 0.0"/>
                 <geometry>
-                    <sphere radius="${wheel_radius}"/>
+                    <cylinder length="${wheel_length}" radius="${wheel_radius}"/>
                 </geometry>
             </collision>

File: pointfoot/WF_TRON1A/xacro/robot.xacro (robot description, xacro)
@@ -28,5 +28,5 @@
         </visual>
         <collision>
-            <origin rpy="0 0 0" xyz="0 0 ${base_height/2}"/>
+            <origin rpy="0 0 0" xyz="0.033 0 -0.07"/>
             <geometry>
                 <box size="${base_length} ${base_width} ${base_height}"/>
@@ -111,5 +111,5 @@
             <origin rpy="1.5707963267948966 0 1.5707963267948966" xyz="0.0149 -0.0175 0"/>
             <geometry>
-                <mesh filename="package://robot_description/pointfoot/meshes_camera/d435.dae"/>
+                <mesh filename="$(find robot_description)/pointfoot/meshes_camera/d435.dae"/>
             </geometry>
         </visual>

File: pointfoot/WF_TRON1A/xacro/ros2_control_interface.xacro (robot description, xacro)
@@ -61,4 +61,27 @@
                     <param name="min">-80</param>
                     <param name="max">80</param>
+                </command_interface>
+                <command_interface name="Kp">
+                    <param name="min">0</param>
+                </command_interface>
+                <command_interface name="Kd">
+                    <param name="min">0</param>
+                </command_interface>
+                <state_interface name="position"/>
+                <state_interface name="velocity"/>
+                <state_interface name="effort"/>
+            </joint>
+            <joint name="wheel_${leg_name}_joint">
+                <command_interface name="position">
+                    <param name="min">-10000000000</param>
+                    <param name="max">10000000000</param>
+                </command_interface>
+                <command_interface name="velocity">
+                    <param name="min">-40</param>
+                    <param name="max">40</param>
+                </command_interface>
+                <command_interface name="effort">
+                    <param name="min">-40</param>
+                    <param name="max">40</param>
                 </command_interface>
                 <command_interface name="Kp">
@@ -143,4 +166,27 @@
                 <state_interface name="effort"/>
             </joint>
+            <joint name="wheel_${leg_name}_joint">
+                <command_interface name="position">
+                    <param name="min">-10000000000</param>
+                    <param name="max">10000000000</param>
+                </command_interface>
+                <command_interface name="velocity">
+                    <param name="min">-40</param>
+                    <param name="max">40</param>
+                </command_interface>
+                <command_interface name="effort">
+                    <param name="min">-40</param>
+                    <param name="max">40</param>
+                </command_interface>
+                <command_interface name="Kp">
+                    <param name="min">0</param>
+                </command_interface>
+                <command_interface name="Kd">
+                    <param name="min">0</param>
+                </command_interface>
+                <state_interface name="position"/>
+                <state_interface name="velocity"/>
+                <state_interface name="effort"/>
+            </joint>
         </xacro:if>
     </xacro:macro>

File: pointfoot/WF_TRON1A/xacro/transmission.xacro (robot description, xacro)
@@ -32,4 +32,14 @@
             </actuator>
         </transmission>
+        <transmission name="wheel_${name}_joint_tran">
+            <type>transmission_interface/SimpleTransmission</type>
+            <joint name="wheel_${name}_joint">
+            <hardwareInterface>hardware_interface/EffortJointInterface</hardwareInterface>
+            </joint>
+            <actuator name="wheel_${name}_joint_motor">
+            <hardwareInterface>hardware_interface/EffortJointInterface</hardwareInterface>
+            <mechanicalReduction>1</mechanicalReduction>
+            </actuator>
+        </transmission>
     </xacro:macro>
 </robot>
