Commit message: 1.1.5.20241216094711

File: pointfoot/WF_TRON1A/urdf/robot.urdf (robot description, URDF)
Before this commit: robot wheel_biped, 10 links, 9 joints
Joints:
- joint abad_L_Joint: limit lower=-0.38397 upper=1.39626 effort=80.0 velocity=20.0 -> lower=-0.38397 upper=1.39626 effort=80.0 velocity=15.0
- joint abad_R_Joint: limit lower=-1.39626 upper=0.38397 effort=80.0 velocity=20.0 -> lower=-1.39626 upper=0.38397 effort=80.0 velocity=15.0
- joint hip_L_Joint: limit lower=-1.012291 upper=1.396263 effort=80.0 velocity=20.0 -> lower=-1.012291 upper=1.396263 effort=80.0 velocity=15.0
- joint hip_R_Joint: limit lower=-1.396263 upper=1.012291 effort=80.0 velocity=20.0 -> lower=-1.396263 upper=1.012291 effort=80.0 velocity=15.0
- joint knee_L_Joint: limit lower=-0.872665 upper=1.361357 effort=80 velocity=20 -> lower=-0.872665 upper=1.361357 effort=80 velocity=15
- joint knee_R_Joint: limit lower=-1.361357 upper=0.872665 effort=80 velocity=20 -> lower=-1.361357 upper=0.872665 effort=80 velocity=15

File: pointfoot/WF_TRON1A/xacro/gazebo.xacro (robot description, xacro)
@@ -84,5 +84,5 @@
         <kd value="100.0"/>
     </gazebo>
-    <gazebo reference="foot_L_Link">
+    <gazebo reference="wheel_L_Link">
         <mu1>2.0</mu1>
         <mu2>2.0</mu2>
@@ -111,5 +111,5 @@
         <kd value="100.0"/>
     </gazebo>
-    <gazebo reference="foot_R_Link">
+    <gazebo reference="wheel_R_Link">
         <mu1>2.0</mu1>
         <mu2>2.0</mu2>
