Commit message: 1.1.5.20241218161059

File: pointfoot/SF_TRON1A/xacro/gazebo.xacro (robot description, xacro)
@@ -35,5 +35,24 @@
         </plugin>
     </gazebo> -->
-    <gazebo reference="imu_Link">
+    <gazebo>
+        <plugin filename="libpointfoot_hw_sim.so" name="gazebo_ros_control">
+            <robotNamespace>/</robotNamespace>
+            <robotParam>robot_description</robotParam>
+            <robotSimType>pointfoot_gazebo/PointFootHWSim</robotSimType>
+        </plugin>
+    </gazebo>
+    <gazebo>
+        <plugin filename="libgazebo_ros_p3d.so" name="p3d_base_controller">
+            <alwaysOn>true</alwaysOn>
+            <updateRate>1000.0</updateRate>
+            <bodyName>base_Link</bodyName>
+            <topicName>ground_truth/state</topicName>
+            <gaussianNoise>0</gaussianNoise>
+            <frameName>world</frameName>
+            <xyzOffsets>0 0 0</xyzOffsets>
+            <rpyOffsets>0 0 0</rpyOffsets>
+        </plugin>
+    </gazebo>
+    <gazebo reference="limx_imu">
         <gravity>true</gravity>
         <sensor name="imu_sensor" type="imu">
@@ -44,24 +63,14 @@
             <plugin filename="libgazebo_ros_imu_sensor.so" name="imu_plugin">
                 <topicName>trunk_imu</topicName>
-                <bodyName>imu_Link</bodyName>
+                <bodyName>limx_imu</bodyName>
                 <updateRateHZ>400.0</updateRateHZ>
                 <gaussianNoise>0.0</gaussianNoise>
                 <xyzOffset>0 0 0</xyzOffset>
                 <rpyOffset>0 0 0</rpyOffset>
-                <frameName>imu_Link</frameName>
+                <frameName>limx_imu</frameName>
                 <initial_orientation_as_reference>false</initial_orientation_as_reference>
             </plugin>
             <pose>0 0 0 0 0 0</pose>
         </sensor>
-    </gazebo>
-    <gazebo reference="stick_link">
-        <mu1>0.2</mu1>
-        <mu2>0.2</mu2>
-        <material>Gazebo/White</material>
-    </gazebo>
-    <gazebo reference="imu_Link">
-        <mu1>0.2</mu1>
-        <mu2>0.2</mu2>
-        <material>Gazebo/Red</material>
     </gazebo>
     <!-- Left leg -->

File: pointfoot/SF_TRON1A/xacro/robot.xacro (robot description, xacro)
@@ -19,4 +19,35 @@
         </joint>
     </xacro:if>
+    <joint name="limx_imu_joint" type="fixed">
+    <parent link="base_Link"/>
+    <child link="limx_imu"/>
+    <origin rpy="0 0 0" xyz="0 0 0"/>
+  </joint>
+  <link name="limx_imu">
+    <inertial>
+      <mass value="0.001"/>
+      <origin rpy="0 0 0" xyz="0 0 0"/>
+      <inertia ixx="0.0001" ixy="0" ixz="0" iyy="0.0001" iyz="0" izz="0.0001"/>
+    </inertial>
+    <visual>
+      <origin rpy="0 0 0" xyz="0 0 0"/>
+      <geometry>
+        <box size="0.015 0.015 0.004"/>
+      </geometry>
+      <material name="red"/>
+    </visual>
+    <collision>
+      <origin rpy="0 0 0" xyz="0 0 0"/>
+      <geometry>
+        <box size=".001 .001 .001"/>
+      </geometry>
+    </collision>
+  </link>
+  <gazebo reference="limx_imu">
+        <material>Gazebo/Orange</material>
+    </gazebo>
+    <gazebo reference="limx_imu_joint">
+        <disableFixedJointLumping>true</disableFixedJointLumping>
+    </gazebo>
     <link name="base_Link">
         <visual>

File: pointfoot/SF_TRON1A/xacro/ros2_control_interface.xacro (robot description, xacro)
@@ -74,6 +74,6 @@
             <joint name="ankle_${leg_name}_joint">
                 <command_interface name="position">
-                    <param name="min">-10000000000</param>
-                    <param name="max">10000000000</param>
+                    <param name="min">-66</param>
+                    <param name="max">90</param>
                 </command_interface>
                 <command_interface name="velocity">
@@ -168,6 +168,6 @@
             <joint name="ankle_${leg_name}_joint">
                 <command_interface name="position">
-                    <param name="min">-10000000000</param>
-                    <param name="max">10000000000</param>
+                    <param name="min">-66</param>
+                    <param name="max">90</param>
                 </command_interface>
                 <command_interface name="velocity">
