Commit message: 3.0.17.20250710121954

File: pointfoot/PF_P441C/urdf/robot.urdf (robot description, URDF)
Before this commit: robot point_foot, 12 links, 11 joints
Joints:
- joint abad_R_Joint: origin xyz=0.039 -0.1095 -0.08725 rpy=0 0 0 -> xyz=0.039 -0.1005 -0.08725 rpy=0 0 0

File: pointfoot/PF_P441C/xacro/const.xacro (robot description, xacro)
@@ -18,5 +18,5 @@
     <!-- abad offset from base frame value -->
     <xacro:property name="abad_offset_x" value="0.039"/>
-    <xacro:property name="abad_offset_y" value="0.1095"/>
+    <xacro:property name="abad_offset_y" value="0.105"/>
     <xacro:property name="abad_offset_z" value="-0.08725"/>
     <!-- hip offset from abad frame value -->

File: pointfoot/PF_P441C/xacro/leg.xacro (robot description, xacro)
@@ -5,5 +5,5 @@
         <joint name="abad_${name}_joint" type="revolute">
             <origin
-                xyz="${abad_offset_x} ${abad_offset_y*mirror} ${abad_offset_z}"
+                xyz="${abad_offset_x} ${(abad_offset_y+0.0045*mirror)*mirror} ${abad_offset_z}"
                 rpy="0 0 0"/>
             <parent link="base_Link"/>
